File: hardware/press-beta.kicad_pcb (KiCad board)
At the start: 2 copper layers, 81.3 x 129.6 mm, 28 parts, among them SW1 SW_Push_45deg, SW10 SW_Push_45deg, SW11 SW_Push_45deg, SW12 SW_Push_45deg, SW13 SW_Push_45deg, SW14 SW_Push_45deg, SW15 SW_Push_45deg, SW16 SW_Push_45deg, SW17 SW_Push_45deg, SW18 SW_Push_45deg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

Commit message: pcb mod
Parts:
- added J1: AudioJack4_SwitchTR1, Connector_Audio:Jack_3.5mm_PJ311_Horizontal, B.Cu at (107.0, 63.1)
- added Q1: PSMN2R0-25MLDX, Package_TO_SOT_SMD:LFPAK33, B.Cu at (85.7, 76.4)
- BT1: footprint Battery:BatteryHolder_TruPower_BH-331P_3xAA -> Connector_Wire:SolderWire-0.75sqmm_1x02_P4.8mm_D1.25mm_OD2.3mm
- U2: footprint Library:LCD -> Library:LCD_nopost
- moved BT1 72.0 mm to (97.8, 76.2), turned to 180 degrees
- moved D1 32.1 mm to (106.7, 76.2), turned to 180 degrees
Connections:
- U1 pad 1: unconnected-(U1-GPIO0-Pad1) -> Net-(U1-GPIO0)
- U1 pad 10: /mosi -> /col2
- U1 pad 11: /miso -> /col3
- U1 pad 12: /clk -> /col4
- U1 pad 13: unconnected-(U1-GND-Pad13) -> GND
- U1 pad 14: /col1 -> unconnected-(U1-GPIO10-Pad14)
- U1 pad 15: /col2 -> unconnected-(U1-GPIO11-Pad15)
- U1 pad 16: /col3 -> unconnected-(U1-GPIO12-Pad16)
- U1 pad 17: /col4 -> Net-(U1-GPIO13)
- U1 pad 18: unconnected-(U1-GND-Pad18) -> GND
- U1 pad 2: unconnected-(U1-GPIO1-Pad2) -> Net-(U1-GPIO1)
- U1 pad 29: unconnected-(U1-GPIO22-Pad29) -> Net-(Q1-G)
- U1 pad 31: unconnected-(U1-GPIO26_ADC0-Pad31) -> Net-(U1-GPIO26_ADC0)
- U1 pad 32: unconnected-(U1-GPIO27_ADC1-Pad32) -> Net-(U1-GPIO27_ADC1)
- U1 pad 33: unconnected-(U1-AGND-Pad33) -> Net-(U1-AGND)
- U1 pad 34: unconnected-(U1-GPIO28_ADC2-Pad34) -> Net-(U1-GPIO28_ADC2)
- U1 pad 4: unconnected-(U1-GPIO2-Pad4) -> /clk
- U1 pad 42: unconnected-(U1-GND-Pad42) -> GND
- U1 pad 5: unconnected-(U1-GPIO3-Pad5) -> /mosi
- U1 pad 6: unconnected-(U1-GPIO4-Pad6) -> /miso
- U1 pad 7: unconnected-(U1-GPIO5-Pad7) -> Net-(U1-GPIO5)
- U1 pad 8: unconnected-(U1-GND-Pad8) -> GND
- U1 pad 9: unconnected-(U1-GPIO6-Pad9) -> /col1
- U2 pad 10: unconnected-(U2-RS-Pad10) -> Net-(U1-GPIO1)
- U2 pad 11: unconnected-(U2-~RESET-Pad11) -> Net-(U1-GPIO0)
- U2 pad 12: unconnected-(U2-~CS-Pad12) -> Net-(U1-GPIO5)
- U2 pad 4: unconnected-(U2-~ROM_CS-Pad4) -> Net-(U1-GPIO13)
- U2 pad 5: +3V3 -> Net-(Q1-S)
Routing:
- net Net-(Q1-G): track 0.00 -> 55.3 mm, vias 0 -> 1
- net Net-(U1-GPIO5): track 0.00 -> 54.6 mm
- net +3V3: track 53.9 -> 0.00 mm
- net Net-(U1-GPIO0): track 0.00 -> 47.8 mm
- net Net-(U1-GPIO13): track 0.00 -> 47.1 mm, vias 0 -> 1
- net Net-(U1-GPIO1): track 0.00 -> 43.5 mm
- net Net-(U1-AGND): track 0.00 -> 39.6 mm, vias 0 -> 2
- net Net-(U1-GPIO26_ADC0): track 0.00 -> 38.5 mm, vias 0 -> 2
- net Net-(U1-GPIO27_ADC1): track 0.00 -> 37.0 mm, vias 0 -> 2
- net Net-(U1-GPIO28_ADC2): track 0.00 -> 35.8 mm
- net Net-(D1-K): track 3.59 -> 34.9 mm, vias 0 -> 1
- net Net-(BT1-+): track 0.00 -> 20.8 mm
- net /col1: track 97.9 -> 116.5 mm
- net /col3: track 105.0 -> 121.5 mm
- net /col2: track 125.7 -> 136.8 mm
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Other:
- board text added: "GTO"
- board text added: "LBL"
- board text added: "P/R"
- board text added: "R/S"
- board text added: "RCL"
- board text added: "STO"
- board text added: "↑"
- board text removed: "CUT"
- board text removed: "PASTE"
- board text removed: "^"

Commit message: lcd working pretty well now
Parts:
- Q1: value PSMN2R0-25MLDX -> AO3400; footprint Package_TO_SOT_SMD:LFPAK33 -> Package_TO_SOT_SMD:SOT-23_Handsoldering
- moved Q1 1.01 mm to (86.6, 75.9), turned to 0 degrees
Routing:
- net Net-(BT1-+): track 20.8 -> 17.6 mm
- net Net-(Q1-G): track 55.3 -> 57.7 mm
Changed lines of the file:
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@@
     )
   )
-  (footprint "Package_TO_SOT_SMD:LFPAK33" (layer "B.Cu")
-    (at 85.734 76.415 -90)
-    (descr "LFPAK33 SOT-1210 https://assets.nexperia.com/documents/outline-drawing/SOT1210.pdf")
-    (tags "LFPAK33 SOT-1210")
+  (footprint "Package_TO_SOT_SMD:SOT-23_Handsoldering" (layer "B.Cu")
+    (at 86.59 75.88)
+    (descr "SOT-23, Handsoldering")
+    (tags "SOT-23")
     (property "Sheetfile" "press-beta.kicad_sch")
     (property "Sheetname" "")
@@
     (property "ki_description" "N-MOSFET transistor, drain/source/gate")
     (property "ki_keywords" "transistor NMOS N-MOS N-MOSFET simulation")
-    (solder_mask_margin 0.05)
     (attr smd)
-    (fp_text reference "Q1" (at 0 2.55 90) (layer "B.SilkS")
+    (fp_text reference "Q1" (at 0 2.5) (layer "B.SilkS")
         (effects (font (size 1 1) (thickness 0.15)) (justify mirror))
     )
-    (fp_text value "PSMN2R0-25MLDX" (at 0 -2.64 90) (layer "B.Fab")
+    (fp_text value "AO3400" (at 0 -2.5) (layer "B.Fab")
         (effects (font (size 1 1) (thickness 0.15)) (justify mirror))
     )
-    (fp_text user "${REFERENCE}" (at 0 0) (layer "B.Fab")
-        (effects (font (size 0.75 0.75) (thickness 0.13)) (justify mirror))
+    (fp_text user "${REFERENCE}" (at 0 0 90) (layer "B.Fab")
+        (effects (font (size 0.5 0.5) (thickness 0.075)) (justify mirror))
     )
-    (fp_line (start -1.95 1.475) (end -1.22 1.475)
+    (fp_line (start 0.76 -1.58) (end -0.7 -1.58)
       (stroke (width 0.12) (type solid)) (layer "B.SilkS"))
-    (fp_line (start -1.22 -1.77) (end 1.62 -1.77)
+    (fp_line (start 0.76 -1.58) (end 0.76 -0.65)
       (stroke (width 0.12) (type solid)) (layer "B.SilkS"))
-    (fp_line (start -1.22 -1.475) (end -1.22 -1.77)
+    (fp_line (start 0.76 1.58) (end -2.4 1.58)
       (stroke (width 0.12) (type solid)) (layer "B.SilkS"))
-    (fp_line (start -1.22 1.77) (end -1.22 1.475)
+    (fp_line (start 0.76 1.58) (end 0.76 0.65)
       (stroke (width 0.12) (type solid)) (layer "B.SilkS"))
-    (fp_line (start 1.62 -1.77) (end 1.62 -1.475)
-      (stroke (width 0.12) (type solid)) (layer "B.SilkS"))
-    (fp_line (start 1.62 1.475) (end 1.62 1.77)
-      (stroke (width 0.12) (type solid)) (layer "B.SilkS"))
-    (fp_line (start 1.62 1.77) (end -1.22 1.77)
-      (stroke (width 0.12) (type solid)) (layer "B.SilkS"))
-    (fp_line (start -2.2 -1.9) (end -2.2 1.9)
+    (fp_line (start -2.7 -1.75) (end -2.7 1.75)
       (stroke (width 0.05) (type solid)) (layer "B.CrtYd"))
-    (fp_line (start -2.2 -1.9) (end 2.2 -1.9)
+    (fp_line (start -2.7 1.75) (end 2.7 1.75)
       (stroke (width 0.05) (type solid)) (layer "B.CrtYd"))
-    (fp_line (start -2.2 1.9) (end 2.2 1.9)
+    (fp_line (start 2.7 -1.75) (end -2.7 -1.75)
       (stroke (width 0.05) (type solid)) (layer "B.CrtYd"))
-    (fp_line (start 2.2 1.9) (end 2.2 -1.9)
+    (fp_line (start 2.7 1.75) (end 2.7 -1.75)
       (stroke (width 0.05) (type solid)) (layer "B.CrtYd"))
-    (fp_line (start -1.1 -1.65) (end 1.5 -1.65)
+    (fp_line (start -0.7 -1.52) (end 0.7 -1.52)
       (stroke (width 0.1) (type solid)) (layer "B.Fab"))
-    (fp_line (start -1.1 1.15) (end -1.1 -1.65)
+    (fp_line (start -0.7 0.95) (end -0.7 -1.5)
       (stroke (width 0.1) (type solid)) (layer "B.Fab"))
-    (fp_line (start -0.6 1.65) (end -1.1 1.15)
+    (fp_line (start -0.7 0.95) (end -0.15 1.52)
       (stroke (width 0.1) (type solid)) (layer "B.Fab"))
-    (fp_line (start -0.6 1.65) (end 1.5 1.65)
+    (fp_line (start -0.15 1.52) (end 0.7 1.52)
       (stroke (width 0.1) (type solid)) (layer "B.Fab"))
-    (fp_line (start 1.5 -1.65) (end 1.5 1.65)
+    (fp_line (start 0.7 1.52) (end 0.7 -1.52)
       (stroke (width 0.1) (type solid)) (layer "B.Fab"))
-    (pad "" smd rect (at -1.535 -0.975 270) (size 0.83 0.3) (layers "B.Paste"))
-    (pad "" smd rect (at -1.535 -0.325 270) (size 0.83 0.3) (layers "B.Paste"))
-    (pad "" smd rect (at -1.535 0.325 270) (size 0.83 0.3) (layers "B.Paste"))
-    (pad "" smd rect (at -1.535 0.975 270) (size 0.83 0.3) (layers "B.Paste"))
-    (pad "" smd rect (at -0.215 -0.626 270) (size 0.51 0.635) (layers "B.Paste"))
-    (pad "" smd rect (at -0.215 0.626 270) (size 0.51 0.635) (layers "B.Paste"))
-    (pad "" smd rect (at 0.645 -0.626 270) (size 0.51 0.635) (layers "B.Paste"))
-    (pad "" smd rect (at 0.645 0.626 270) (size 0.51 0.635) (layers "B.Paste"))
-    (pad "" smd rect (at 1.575 -0.975 270) (size 0.75 0.3) (layers "B.Paste"))
-    (pad "" smd rect (at 1.575 -0.325 270) (size 0.75 0.3) (layers "B.Paste"))
-    (pad "" smd rect (at 1.575 0.325 270) (size 0.75 0.3) (layers "B.Paste"))
-    (pad "" smd rect (at 1.575 0.975 270) (size 0.75 0.3) (layers "B.Paste"))
-    (pad "1" smd custom (at 0.405 0 270) (size 1.85 2.25) (layers "B.Cu" "B.Mask")
-      (net 1 "Net-(BT1-+)") (pinfunction "D") (pintype "passive") (zone_connect 2) (thermal_bridge_angle 45)
-      (options (clearance outline) (anchor rect))
-      (primitives
-        (gr_poly
-          (pts
-            (xy 1.545 0.775)
-            (xy 0.925 0.775)
-            (xy 0.925 1.175)
-            (xy 1.545 1.175)
-          )
-          (width 0) (fill yes))
-        (gr_poly
-          (pts
-            (xy 1.545 0.125)
-            (xy 0.925 0.125)
-            (xy 0.925 0.525)
-            (xy 1.545 0.525)
-          )
-          (width 0) (fill yes))
-        (gr_poly
-          (pts
-            (xy 1.545 -0.525)
-            (xy 0.925 -0.525)
-            (xy 0.925 -0.125)
-            (xy 1.545 -0.125)
-          )
-          (width 0) (fill yes))
-        (gr_poly
-          (pts
-            (xy 1.545 -1.175)
-            (xy 0.925 -1.175)
-            (xy 0.925 -0.775)
-            (xy 1.545 -0.775)
-          )
-          (width 0) (fill yes))
-      ))
-    (pad "2" smd rect (at -1.535 -0.975 270) (size 0.83 0.4) (layers "B.Cu" "B.Mask")
+    (pad "1" smd rect (at 1.5 0) (size 1.9 0.8) (layers "B.Cu" "B.Paste" "B.Mask")
+      (net 1 "Net-(BT1-+)") (pinfunction "D") (pintype "passive"))
+    (pad "2" smd rect (at -1.5 0.95) (size 1.9 0.8) (layers "B.Cu" "B.Paste" "B.Mask")
       (net 10 "Net-(Q1-G)") (pinfunction "G") (pintype "input"))
-    (pad "3" smd rect (at -1.535 -0.325 270) (size 0.83 0.4) (layers "B.Cu" "B.Mask")
-      (net 14 "Net-(Q1-S)") (pinfunction "S") (pintype "passive"))
-    (pad "3" smd rect (at -1.535 0.325 270) (size 0.83 0.4) (layers "B.Cu" "B.Mask")
-      (net 14 "Net-(Q1-S)") (pinfunction "S") (pintype "passive"))
-    (pad "3" smd rect (at -1.535 0.975 270) (size 0.83 0.4) (layers "B.Cu" "B.Mask")
+    (pad "3" smd rect (at -1.5 -0.95) (size 1.9 0.8) (layers "B.Cu" "B.Paste" "B.Mask")
       (net 14 "Net-(Q1-S)") (pinfunction "S") (pintype "passive"))
-    (model "${KICAD6_3DMODEL_DIR}/Package_TO_SOT_SMD.3dshapes/LFPAK33.wrl"
+    (model "${KICAD6_3DMODEL_DIR}/Package_TO_SOT_SMD.3dshapes/SOT-23.wrl"
       (offset (xyz 0 0 0))
       (scale (xyz 1 1 1))
@@
     )
   )
-  (segment (start 95.25 73.66) (end 97.79 76.2) (width 1) (layer "B.Cu") (net 1))
-  (segment (start 89.9504 73.66) (end 95.25 73.66) (width 1) (layer "B.Cu") (net 1))
-  (segment (start 85.734 76.82) (end 86.7904 76.82) (width 1) (layer "B.Cu") (net 1))
+  (segment (start 95.8118 74.2218) (end 97.79 76.2) (width 1) (layer "B.Cu") (net 1))
+  (segment (start 88.09 75.88) (end 89.7482 74.2218) (width 1) (layer "B.Cu") (net 1))
+  (segment (start 89.7482 74.2218) (end 95.8118 74.2218) (width 1) (layer "B.Cu") (net 1))
   (segment (start 97.79 76.2) (end 104.22 76.2) (width 1) (layer "B.Cu") (net 1))
-  (segment (start 86.7904 76.82) (end 89.9504 73.66) (width 1) (layer "B.Cu") (net 1))
   (segment (start 74.1 67.61) (end 78.21 63.5) (width 0.25) (layer "B.Cu") (net 3))
   (segment (start 115.6618 59.5982) (end 115.6618 58.3282) (width 0.25) (layer "B.Cu") (net 3))
@@
   (segment (start 118.122393 71.120136) (end 120.650136 71.120136) (width 0.25) (layer "F.Cu") (net 10))
   (via (at 118.122393 71.120136) (size 0.8) (drill 0.4) (layers "F.Cu" "B.Cu") (net 10))
-  (segment (start 86.709 74.7305) (end 90.3195 71.12) (width 0.25) (layer "B.Cu") (net 10))
-  (segment (start 86.709 74.88) (end 86.709 74.7305) (width 0.25) (layer "B.Cu") (net 10))
-  (segment (start 90.3195 71.12) (end 118.122257 71.12) (width 0.25) (layer "B.Cu") (net 10))
-  (segment (start 118.122257 71.12) (end 118.122393 71.120136) (width 0.25) (layer "B.Cu") (net 10))
+  (segment (start 90.8 71.12) (end 85.09 76.83) (width 0.25) (layer "B.Cu") (net 10))
+  (segment (start 118.122393 71.120136) (end 118.122257 71.12) (width 0.25) (layer "B.Cu") (net 10))
+  (segment (start 118.122257 71.12) (end 90.8 71.12) (width 0.25) (layer "B.Cu") (net 10))
   (segment (start 82.02 64.77) (end 96.66 64.77) (width 0.25) (layer "B.Cu") (net 11))
   (segment (start 101.6 68.58) (end 101.9082 68.8882) (width 0.25) (layer "B.Cu") (net 11))

Commit message: first hardware iteration?
Parts:
- added G***: LOGO, LOGO, B.Cu at (101.6, 148.6)
Routing:
- net +3V3: track 0.00 -> 69.4 mm
- net Net-(U1-GPIO13): track 47.1 -> 45.7 mm
Other:
- board text added: "A"
- board text added: "B"
- board text added: "C"
- board text added: "D"
- board text added: "E"
- board text added: "F"
- board text added: "G"
- board text added: "H"
- board text added: "J"
- board text added: "L"
- board text added: "M"
- board text added: "MAHIRO1"
- board text added: "N"
- board text added: "P"
- board text added: "Q"
- board text added: "R"
- board text added: "T"
- board text added: "U"
- board text added: "V"
- board text added: "W"
- board text added: "X"
- board text added: "Y"
- board text added: "Z"
- board text added: "η↑"
- board text added: "η↓"
